Commit message: feat(PR-687): simplify urdf head base collider

File: mujoco/pib_head_only.urdf (robot description, URDF)
Before this commit: robot pib, 4 links, 3 joints
Links:
- link urdf_head_base: geometry collision box size=0.11000000000000000056 0.092999999999999999334 0.0299999999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; visual mesh filename=package://pib_head_module/urdf_head_base.stl
