Commit message: feat(PR-687): update upper body urdf with simplified colliders

File: mujoco/pib_upper_body/pib_upper_body.urdf (robot description, URDF)
Before this commit: robot pib, 39 links, 38 joints
Links:
- link urdf_body: geometry collision box size=0.26900000000000001688 0.12679999999999999605 0.31400000000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; collision box size=0.26900000000000001688 0.17780000000000001359 0.27400000000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
- link urdf_elbow-lower: geometry collision cylinder length=0.064000000000000001332 radius=0.044999999999999998335; visual mesh filename=package://pib_head_module/meshes/urdf_elbow-lower.stl
- link urdf_elbow-lower_2: geometry collision cylinder length=0.064000000000000001332 radius=0.044999999999999998335; visual mesh filename=package://pib_head_module/meshes/urdf_elbow-lower.stl
- link urdf_elbow-upper: geometry collision cylinder length=0.067000000000000003997 radius=0.044999999999999998335; visual mesh filename=package://pib_head_module/meshes/urdf_elbow-upper.stl
- link urdf_elbow-upper_2: geometry collision cylinder length=0.067000000000000003997 radius=0.044999999999999998335; visual mesh filename=package://pib_head_module/meshes/urdf_elbow-upper.stl
- link urdf_finger_distal: geometry collision cylinder length=0.044999999999999998335 radius=0.0080000000000000001665; visual mesh filename=package://pib_head_module/meshes/urdf_finger_distal.stl
- link urdf_finger_distal_10: geometry collision cylinder length=0.044999999999999998335 radius=0.0080000000000000001665; visual mesh filename=package://pib_head_module/meshes/urdf_finger_distal.stl
- link urdf_finger_distal_2: geometry collision cylinder length=0.044999999999999998335 radius=0.0080000000000000001665; visual mesh filename=package://pib_head_module/meshes/urdf_finger_distal.stl
- link urdf_finger_distal_3: geometry collision cylinder length=0.044999999999999998335 radius=0.0080000000000000001665; visual mesh filename=package://pib_head_module/meshes/urdf_finger_distal.stl
- link urdf_finger_distal_4: geometry collision cylinder length=0.044999999999999998335 radius=0.0080000000000000001665; visual mesh filename=package://pib_head_module/meshes/urdf_finger_distal.stl
- link urdf_finger_distal_5: geometry collision cylinder length=0.044999999999999998335 radius=0.0080000000000000001665; visual mesh filename=package://pib_head_module/meshes/urdf_finger_distal.stl
- link urdf_finger_distal_6: geometry collision cylinder length=0.044999999999999998335 radius=0.0080000000000000001665; visual mesh filename=package://pib_head_module/meshes/urdf_finger_distal.stl
- link urdf_finger_distal_7: geometry collision cylinder length=0.044999999999999998335 radius=0.0080000000000000001665; visual mesh filename=package://pib_head_module/meshes/urdf_finger_distal.stl
- link urdf_finger_distal_8: geometry collision cylinder length=0.044999999999999998335 radius=0.0080000000000000001665; visual mesh filename=package://pib_head_module/meshes/urdf_finger_distal.stl
- link urdf_finger_distal_9: geometry collision cylinder length=0.044999999999999998335 radius=0.0080000000000000001665; visual mesh filename=package://pib_head_module/meshes/urdf_finger_distal.stl
- link urdf_finger_proximal: geometry collision cylinder length=0.037999999999999999056 radius=0.00899999999999999932; visual mesh filename=package://pib_head_module/meshes/urdf_finger_proximal.stl
- link urdf_finger_proximal_10: geometry collision cylinder length=0.037999999999999999056 radius=0.00899999999999999932; visual mesh filename=package://pib_head_module/meshes/urdf_finger_proximal.stl
- link urdf_finger_proximal_2: geometry collision cylinder length=0.037999999999999999056 radius=0.00899999999999999932; visual mesh filename=package://pib_head_module/meshes/urdf_finger_proximal.stl
- link urdf_finger_proximal_3: geometry collision cylinder length=0.037999999999999999056 radius=0.00899999999999999932; visual mesh filename=package://pib_head_module/meshes/urdf_finger_proximal.stl
- link urdf_finger_proximal_4: geometry collision cylinder length=0.037999999999999999056 radius=0.00899999999999999932; visual mesh filename=package://pib_head_module/meshes/urdf_finger_proximal.stl
- link urdf_finger_proximal_5: geometry collision cylinder length=0.037999999999999999056 radius=0.00899999999999999932; visual mesh filename=package://pib_head_module/meshes/urdf_finger_proximal.stl
- link urdf_finger_proximal_6: geometry collision cylinder length=0.037999999999999999056 radius=0.00899999999999999932; visual mesh filename=package://pib_head_module/meshes/urdf_finger_proximal.stl
- link urdf_finger_proximal_7: geometry collision cylinder length=0.037999999999999999056 radius=0.00899999999999999932; visual mesh filename=package://pib_head_module/meshes/urdf_finger_proximal.stl
- link urdf_finger_proximal_8: geometry collision cylinder length=0.037999999999999999056 radius=0.00899999999999999932; visual mesh filename=package://pib_head_module/meshes/urdf_finger_proximal.stl
- link urdf_finger_proximal_9: geometry collision cylinder length=0.037999999999999999056 radius=0.00899999999999999932; visual mesh filename=package://pib_head_module/meshes/urdf_finger_proximal.stl
- link urdf_forearm: geometry collision cylinder length=0.13400000000000000799 radius=0.02999999999999999889; visual mesh filename=package://pib_head_module/meshes/urdf_forearm.stl
- link urdf_forearm_2: geometry collision cylinder length=0.13400000000000000799 radius=0.02999999999999999889; visual mesh filename=package://pib_head_module/meshes/urdf_forearm.stl
- link urdf_head: geometry collision box size=0.025000000000000001388 0.15099999999999999534 0.1300000000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; collision box size=0.025000000000000001388 0.15099999999999999534 0.1300000000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
- link urdf_head_base: geometry collision box size=0.080000000000000001665 0.080000000000000001665 0.025000000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; visual mesh filename=package://pib_head_module/meshes/urdf_head_base.stl
- link urdf_palm_left: geometry collision box size=0.02999999999999999889 0.020000000000000000416 0.0500000000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; collision box size=0.050000000000000002776 0.020000000000000000416 0.029999999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
- link urdf_palm_right: geometry collision box size=0.020000000000000000416 0.02999999999999999889 0.0500000000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; collision box size=0.020000000000000000416 0.050000000000000002776 0.029999999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
- link urdf_shoulder_horizontal: geometry collision cylinder length=0.076999999999999999001 radius=0.044999999999999998335; visual mesh filename=package://pib_head_module/meshes/urdf_shoulder_horizontal.s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
- link urdf_shoulder_horizontal_2: geometry collision cylinder length=0.076999999999999999001 radius=0.044999999999999998335; visual mesh filename=package://pib_head_module/meshes/urdf_shoulder_horizontal.s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
- link urdf_shoulder_vertical: geometry collision box size=0.00899999999999999932 0.11000000000000000056 0.10499999999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; visual mesh filename=package://pib_head_module/meshes/urdf_shoulder_vertical.stl
- link urdf_shoulder_vertical_2: geometry collision box size=0.00899999999999999932 0.11000000000000000056 0.10499999999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; visual mesh filename=package://pib_head_module/meshes/urdf_shoulder_vertical.stl
- link urdf_thumb_rotator_left: geometry collision cylinder length=0.034000000000000002442 radius=0.0050000000000000001041; visual mesh filename=package://pib_head_module/meshes/urdf_thumb_rotator_left.stl
- link urdf_thumb_rotator_right: geometry collision cylinder length=0.034000000000000002442 radius=0.0050000000000000001041; visual mesh filename=package://pib_head_module/meshes/urdf_thumb_rotator_right.s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
